Commit message: Add files via upload

File: ruka_description/urdf/gripper_macro.xacro (robot description, xacro)
@@ -1,19 +1,18 @@
 <?xml version="1.0"?>
 <robot xmlns:xacro="http://www.ros.org/wiki/xacro">
-<robot xmlns:xacro="http://ros.org/wiki/xacro">
     <xacro:macro name="gripper_macro" params="prefix">
         <link name="${prefix}gripper">
           <inertial>
               <origin
-                  xyz="-8.0961E-06 0.0019103 0.028995"
+                  xyz="0 0 0"
                   rpy="0 0 0" />
-              <mass value="0.90882" />
+              <mass value="0.5" />
               <inertia
-                  ixx="0.0014545"
-                  ixy="4.2968E-08"
-                  ixz="-1.8199E-07"
-                  iyy="0.001345"
-                  iyz="-6.243E-06"
-                  izz="0.002155" />
+                  ixx="0.0001"
+                  ixy="0"
+                  ixz="0"
+                  iyy="0.0001"
+                  iyz="0"
+                  izz="0.0001" />
           </inertial>
           <visual>
