Commit message: Add files via upload

File: ruka_description/urdf/gripper_bunka.xacro (robot description, xacro)
@@ -2,5 +2,4 @@
 <robot xmlns:xacro="http://www.ros.org/wiki/xacro" name = "cr5_robot">
     <xacro:arg name="arm_id" default="cr5_robot" />
-<!-- include dobot svoj gripper create_joint aby ssa spojil dobot a gripepr -->
     <xacro:include filename="$(find ruka_description)/urdf/dobot_macro.xacro"/>
     <xacro:cr5_robot prefix=""/>
@@ -8,5 +7,5 @@
     <xacro:gripper_macro prefix=""/>
     <joint name="dobot_gripper_joint" type="fixed">
-        <origin xyz="0 0 0" rpy="0 0 -1.57" />
+        <origin xyz="0 0 0" rpy="0 0 0" />
         <parent link="Link6" />
         <child  link="gripper" />

File: ruka_description/urdf/gripper_macro.xacro (robot description, xacro)
@@ -21,5 +21,5 @@
                   rpy="0 0 0" />
               <geometry>
-                  <mesh filename="package://ruka_description/meshes/gripper/Gripper_1.4_mod_s_vzduch_pris.STL" />
+                  <mesh scale = "0.001 0.001 0.001" filename="package://ruka_description/meshes/gripper/Gripper_1.4_mod_s_vzduch_pris.STL" />
               </geometry>
               <material name="">
@@ -32,5 +32,5 @@
                   rpy="0 0 0" />
               <geometry>
-                  <mesh filename="package://ruka_description/meshes/gripper/Gripper_1.4_mod_s_vzduch_pris.STL" />
+                  <mesh scale = "0.001 0.001 0.001" filename="package://ruka_description/meshes/gripper/Gripper_1.4_mod_s_vzduch_pris.STL" />
               </geometry>
           </collision>
