Commit message: Add files via upload

File: ruka_description/urdf/dobot_macro.xacro (robot description, xacro)
@@ -1,9 +1,10 @@
 <?xml version="1.0"?>
 <robot xmlns:xacro="http://www.ros.org/wiki/xacro" name = "cr5_robot">
+<xacro:property name="prefix" value=""/>
 <!--params neviem ci tammaju byt-->
   <xacro:macro name="cr5_robot" params="prefix">
       <!--<link name="dummy_link">
       </link>-->
-      <link name="base_link">
+      <link name="${prefix}base_link">
           <inertial>
               <origin
@@ -39,5 +40,5 @@
           </collision>
       </link>
-      <link name="Link1">
+      <link name="${prefix}Link1">
           <inertial>
               <origin
@@ -73,14 +74,5 @@
           </collision>
       </link>
-      <joint name="joint1" type="revolute">
-          <origin
-              xyz="0 0 0.147"
-              rpy="0 0 0" />
-          <parent link="base_link" />
-          <child link="Link1" />
-          <axis xyz="0 0 1" />
-          <limit lower= "-3.14" upper="3.14" effort="0" velocity="0" />
-      </joint>
-      <link name="Link2">
+      <link name="${prefix}Link2">
           <inertial>
           <origin
@@ -116,14 +108,5 @@
           </collision>
       </link>
-      <joint name="joint2" type="revolute">
-          <origin
-              xyz="0 0 0"
-              rpy="1.5708 1.5708 0" />
-          <parent link="Link1" />
-          <child link="Link2" />
-          <axis xyz="0 0 1" />
-          <limit lower= "-3.14" upper="3.14" effort="0" velocity="0" />
-      </joint>
-      <link name="Link3">
+      <link name="${prefix}Link3">
           <inertial>
               <origin
@@ -159,14 +142,5 @@
           </collision>
       </link>
-      <joint name="joint3" type="revolute">
-          <origin
-              xyz="-0.427 0 0"
-              rpy="0 0 0" />
-          <parent link="Link2" />
-          <child link="Link3" />
-          <axis xyz="0 0 1" />
-          <limit lower= "-2.86"  upper="2.86"  effort="0" velocity="0" />
-      </joint>
-        <link name="Link4">
+        <link name="${prefix}Link4">
             <inertial>
                 <origin
@@ -202,14 +176,5 @@
             </collision>
       </link>
-      <joint name="joint4" type="revolute">
-          <origin
-              xyz="-0.357 0 0.141"
-              rpy="0 0 -1.5708" />
-          <parent link="Link3" />
-          <child link="Link4" />
-          <axis xyz="0 0 1" />
-          <limit lower= "-3.14" upper="3.14" effort="0" velocity="0" />
-      </joint>
-        <link name="Link5">
+        <link name="${prefix}Link5">
             <inertial>
                 <origin
@@ -245,14 +210,5 @@
             </collision>
       </link>
-      <joint name="joint5" type="revolute">
-          <origin
-              xyz="0 -0.116 0"
-              rpy="1.5708 0 0" />
-          <parent link="Link4" />
-          <child link="Link5" />
-          <axis xyz="0 0 1" />
-          <limit lower= "-3.14" upper="3.14" effort="0" velocity="0" />
-      </joint>
-        <link name="Link6">
+        <link name="${prefix}Link6">
             <inertial>
                 <origin
@@ -288,10 +244,55 @@
             </collision>
       </link>
-      <joint name="joint6" type="revolute">
+      <joint name="${prefix}joint1" type="revolute">
+          <origin
+              xyz="0 0 0.147"
+              rpy="0 0 0" />
+          <parent link="${prefix}base_link" />
+          <child link="${prefix}Link1" />
+          <axis xyz="0 0 1" />
+          <limit lower= "-3.14" upper="3.14" effort="0" velocity="0" />
+      </joint>
+      <joint name="${prefix}joint2" type="revolute">
+          <origin
+              xyz="0 0 0"
+              rpy="1.5708 1.5708 0" />
+          <parent link="${prefix}Link1" />
+          <child link="${prefix}Link2" />
+          <axis xyz="0 0 1" />
+          <limit lower= "-3.14" upper="3.14" effort="0" velocity="0" />
+      </joint>
+      <joint name="${prefix}joint3" type="revolute">
+          <origin
+              xyz="-0.427 0 0"
+              rpy="0 0 0" />
+          <parent link="${prefix}Link2" />
+          <child link="${prefix}Link3" />
+          <axis xyz="0 0 1" />
+          <limit lower= "-2.86"  upper="2.86"  effort="0" velocity="0" />
+      </joint>
+      <joint name="${prefix}joint4" type="revolute">
+          <origin
+              xyz="-0.357 0 0.141"
+              rpy="0 0 -1.5708" />
+          <parent link="${prefix}Link3" />
+          <child link="${prefix}Link4" />
+          <axis xyz="0 0 1" />
+          <limit lower= "-3.14" upper="3.14" effort="0" velocity="0" />
+      </joint>
+      <joint name="${prefix}joint5" type="revolute">
+          <origin
+              xyz="0 -0.116 0"
+              rpy="1.5708 0 0" />
+          <parent link="${prefix}Link4" />
+          <child link="${prefix}Link5" />
+          <axis xyz="0 0 1" />
+          <limit lower= "-3.14" upper="3.14" effort="0" velocity="0" />
+      </joint>
+      <joint name="${prefix}joint6" type="revolute">
           <origin
               xyz="0 0.105 0"
               rpy="-1.5708 0 0" />
-          <parent link="Link5" />
-          <child link="Link6" />
+          <parent link="${prefix}Link5" />
+          <child link="${prefix}Link6" />
           <axis xyz="0 0 1" />
           <limit lower= "-6.28" upper="6.28" effort="0" velocity="0" />

Commit message: Add files via upload

File: ruka_description/urdf/dobot_macro.xacro (robot description, xacro)
@@ -1,9 +1,7 @@
 <?xml version="1.0"?>
-<robot xmlns:xacro="http://www.ros.org/wiki/xacro" name = "cr5_robot">
-<xacro:property name="prefix" value=""/>
-<!--params neviem ci tammaju byt-->
+<robot xmlns:xacro="http://www.ros.org/wiki/xacro">
+<!--params neviem ci tammaju byt <xacro:include filename = "cr5_robot">-->
   <xacro:macro name="cr5_robot" params="prefix">
-      <!--<link name="dummy_link">
-      </link>-->
+      <link name="dummy_link"/>
       <link name="${prefix}base_link">
           <inertial>
@@ -40,4 +38,8 @@
           </collision>
       </link>
+      <joint name="${prefix}dummy_joint" type="fixed">
+          <parent link="${prefix}dummy_link" />
+          <child link="${prefix}base_link" />
+      </joint>
       <link name="${prefix}Link1">
           <inertial>

File: ruka_description/urdf/gripper_bunka.xacro (robot description, xacro)
@@ -1 +1,14 @@
-include dobot svoj gripper create_joint aby ssa spojil dobot a gripepr
+<?xml version="1.0"?>
+<robot xmlns:xacro="http://www.ros.org/wiki/xacro" name = "cr5_robot">
+    <xacro:arg name="arm_id" default="cr5_robot" />
+<!-- include dobot svoj gripper create_joint aby ssa spojil dobot a gripepr -->
+    <xacro:include filename="$(find ruka_description)/urdf/dobot_macro.xacro"/>
+    <xacro:cr5_robot prefix=""/>
+    <xacro:include filename="$(find ruka_description)/urdf/gripper_macro.xacro"/>
+    <xacro:gripper_macro prefix=""/>
+    <joint name="dobot_gripper_joint" type="fixed">
+        <origin xyz="0 0 0" rpy="0 0 -1.57" />
+        <parent link="Link6" />
+        <child  link="gripper" />
+    </joint>
+</robot>

Commit message: Add files via upload

File: ruka_description/urdf/dobot_macro.xacro (robot description, xacro)
@@ -3,5 +3,5 @@
 <!--params neviem ci tammaju byt <xacro:include filename = "cr5_robot">-->
   <xacro:macro name="cr5_robot" params="prefix">
-      <link name="dummy_link"/>
+      <link name="${prefix}dummy_link"/>
       <link name="${prefix}base_link">
           <inertial>
